Commit message: cametra traseira

File: parte12/robutler_description/urdf/robutler.gazebo.xacro (robot description, xacro)
@@ -188,5 +188,5 @@
           </clip>
       </camera>
-      <plugin name="camera_controller" filename="libgazebo_ros_camera.so">
+      <plugin name="camera_controller_back" filename="libgazebo_ros_camera.so">
         <alwaysOn>true</alwaysOn>
         <updateRate>30.0</updateRate>

File: parte12/robutler_description/urdf/robutler.urdf.xacro (robot description, xacro)
@@ -189,5 +189,5 @@
   <!-- Camera traseira -->
   <joint name="camera_joint_back" type="fixed">
-    <origin xyz="0.073 -0.011 0.084" rpy="3.14 3.14 3.14"/>
+    <origin xyz="-0.173 -0.011 0.084" rpy="0 0 0"/>
     <parent link="base_link"/>
     <child link="camera_link_back"/>
@@ -195,5 +195,5 @@
   <link name="camera_link_back">
     <collision>
-      <origin xyz="0.005 0.011 0.013" rpy="3.14 3.14 3.14"/>
+      <origin xyz="-0.105 -0.011 0.013" rpy="0 0 0"/>
       <geometry>
         <box size="0.015 0.030 0.027"/>
@@ -202,5 +202,5 @@
   </link>
   <joint name="camera_rgb_joint_back" type="fixed">
-    <origin xyz="0.003 0.011 0.009" rpy="3.14 3.14 3.14"/>
+    <origin xyz="-0.103 -0.011 0.009" rpy="0 0 3.14"/>
     <parent link="camera_link_back"/>
     <child link="camera_rgb_frame_back"/>
@@ -208,5 +208,5 @@
   <link name="camera_rgb_frame_back"/>
   <joint name="camera_rgb_optical_back" type="fixed">
-    <origin xyz="0 0 0" rpy="1.57 0 1.57"/>
+    <origin xyz="0 0 0" rpy="0 0 3.14"/>
     <parent link="camera_rgb_frame_back"/>
     <child link="camera_rgb_optical_back"/>
